File: PWR_Supply/12V.sch (KiCad schematic (older format))
At the start: 3 parts

Commit message: single_amp
Parts:
- gave numbers to parts that had none: 1
- renumbered 0.1uF to 0.1uF7, 0.1uF to 0.1uF8
Changed lines of the file:
@@
 LIBS:contrib
 LIBS:valves
+LIBS:PWR_Supply-cache
 EELAYER 25 0
 EELAYER END
@@
 $EndDescr
 $Comp
-L LM7812ACT U?
+L LM7812ACT U4
 U 1 1 58D2C836
 P 5100 4900
-F 0 "U?" H 4900 5100 50  0000 C CNN
+F 0 "U4" H 4900 5100 50  0000 C CNN
 F 1 "LM7812ACT" H 5100 5100 50  0000 L CNN
 F 2 "TO-220" H 5100 5000 50  0000 C CIN
@@
 $EndComp
 $Comp
-L CP1 0.1uF
+L CP1 0.1uF8
 U 1 1 58D2CE2C
 P 5900 5450
-F 0 "0.1uF" H 5925 5550 50  0000 L CNN
+F 0 "0.1uF8" H 5925 5550 50  0000 L CNN
 F 1 "CP1" H 5925 5350 50  0000 L CNN
 F 2 "" H 5900 5450 50  0000 C CNN
@@
 $EndComp
 $Comp
-L CP1 0.1uF
+L CP1 0.1uF7
 U 1 1 58D2CEE7
 P 4250 5450
-F 0 "0.1uF" H 4275 5550 50  0000 L CNN
+F 0 "0.1uF7" H 4275 5550 50  0000 L CNN
 F 1 "CP1" H 4275 5350 50  0000 L CNN
 F 2 "" H 4250 5450 50  0000 C CNN
