File: PWR_Supply/5V.sch (KiCad schematic (older format))
At the start: 3 parts

Commit message: single_amp
Parts:
- gave numbers to parts that had none: 1
- renumbered 0.1uF to 0.1uF3, 0.1uF to 0.1uF4
Changed lines of the file:
@@
 LIBS:contrib
 LIBS:valves
+LIBS:PWR_Supply-cache
 EELAYER 25 0
 EELAYER END
@@
 $EndDescr
 $Comp
-L 7805 U?
+L 7805 U2
 U 1 1 58D294B5
 P 4900 2450
-F 0 "U?" H 5050 2254 50  0000 C CNN
+F 0 "U2" H 5050 2254 50  0000 C CNN
 F 1 "7805" H 4900 2650 50  0000 C CNN
 F 2 "" H 4900 2450 50  0000 C CNN
@@
 $EndComp
 $Comp
-L CP1 0.1uF
+L CP1 0.1uF3
 U 1 1 58D29578
 P 3700 2900
-F 0 "0.1uF" H 3725 3000 50  0000 L CNN
+F 0 "0.1uF3" H 3725 3000 50  0000 L CNN
 F 1 "CP1" H 3725 2800 50  0000 L CNN
 F 2 "" H 3700 2900 50  0000 C CNN
@@
 $EndComp
 $Comp
-L CP1 0.1uF
+L CP1 0.1uF4
 U 1 1 58D2962C
 P 6000 2950
-F 0 "0.1uF" H 6025 3050 50  0000 L CNN
+F 0 "0.1uF4" H 6025 3050 50  0000 L CNN
 F 1 "CP1" H 6025 2850 50  0000 L CNN
 F 2 "" H 6000 2950 50  0000 C CNN

Commit message: Kursa_darbs_PCB
Parts:
- removed U2: 7805, symbol 7805
- added U2: LM7805CT, TO-220, symbol LM7805CT
Connections:
- net +5V: now also U2.3 (OUT)
- net GND: now also U2.2 (GND)
- net VCC: now also U2.1 (IN)
Changed lines of the file:
@@
 $Descr A4 11693 8268
 encoding utf-8
-Sheet 4 6
+Sheet 3 6
 Title ""
 Date ""
@@
 Comment4 ""
 $EndDescr
-$Comp
-L 7805 U2
-U 1 1 58D294B5
-P 4900 2450
-F 0 "U2" H 5050 2254 50  0000 C CNN
-F 1 "7805" H 4900 2650 50  0000 C CNN
-F 2 "" H 4900 2450 50  0000 C CNN
-F 3 "" H 4900 2450 50  0000 C CNN
-	1    4900 2450
-	1    0    0    -1
-$EndComp
 $Comp
 L CP1 0.1uF3
@@
 $EndComp
 $Comp
-L GND #PWR03
+L GND #PWR04
 U 1 1 58D29684
 P 4900 3400
-F 0 "#PWR03" H 4900 3150 50  0001 C CNN
+F 0 "#PWR04" H 4900 3150 50  0001 C CNN
 F 1 "GND" H 4900 3250 50  0000 C CNN
 F 2 "" H 4900 3400 50  0000 C CNN
@@
 	4900 2700 4900 3400
 Connection ~ 4900 3200
+$Comp
+L LM7805CT U2
+U 1 1 59462669
+P 4900 2450
+F 0 "U2" H 4700 2650 50  0000 C CNN
+F 1 "LM7805CT" H 4900 2650 50  0000 L CNN
+F 2 "TO-220" H 4900 2550 50  0000 C CIN
+F 3 "" H 4900 2450 50  0000 C CNN
+	1    4900 2450
+	1    0    0    -1
+$EndComp
 $EndSCHEMATC
