File: PWR_Supply/9V.sch (KiCad schematic (older format))
At the start: 3 parts

Commit message: single_amp
Parts:
- gave numbers to parts that had none: 1
- renumbered 0.1uF to 0.1uF5, 0.1uF to 0.1uF6
Changed lines of the file:
@@
 LIBS:contrib
 LIBS:valves
+LIBS:PWR_Supply-cache
 EELAYER 25 0
 EELAYER END
@@
 $EndDescr
 $Comp
-L LM7809ACT U?
+L LM7809ACT U3
 U 1 1 58D2A952
 P 4800 2200
-F 0 "U?" H 4600 2400 50  0000 C CNN
+F 0 "U3" H 4600 2400 50  0000 C CNN
 F 1 "LM7809ACT" H 4800 2400 50  0000 L CNN
 F 2 "TO-220" H 4800 2300 50  0000 C CIN
@@
 $EndComp
 $Comp
-L CP1 0.1uF
+L CP1 0.1uF5
 U 1 1 58D2A9DE
 P 3900 2650
-F 0 "0.1uF" H 3925 2750 50  0000 L CNN
+F 0 "0.1uF5" H 3925 2750 50  0000 L CNN
 F 1 "CP1" H 3925 2550 50  0000 L CNN
 F 2 "" H 3900 2650 50  0000 C CNN
@@
 $EndComp
 $Comp
-L CP1 0.1uF
+L CP1 0.1uF6
 U 1 1 58D2AA3D
 P 5650 2600
-F 0 "0.1uF" H 5675 2700 50  0000 L CNN
+F 0 "0.1uF6" H 5675 2700 50  0000 L CNN
 F 1 "CP1" H 5675 2500 50  0000 L CNN
 F 2 "" H 5650 2600 50  0000 C CNN
