File: PWR_Supply/PWR_Supply.sch (KiCad schematic (older format))
At the start: 0 parts

Commit message: Kursa_darbs_PCB
Parts:
- added P2: CONN_01X04, symbol CONN_01X04
Connections:
- net labels added: 1, 2, 3, 4
- wire segments 8 -> 27
Changed lines of the file:
@@
 $EndDescr
 $Sheet
-S 1700 650  2800 1450
+S 4050 900  2800 1450
 U 58D26FA5
 F0 "block_1" 60
 F1 "unstabile.sch" 60
-F2 "VCC" I L 1700 950 60
-F3 "GND" I L 1700 1850 60
+F2 "GND" I L 4050 2100 60
+F3 "VCC" O R 6850 1150 60
+F4 "220V_IN" I L 4050 1100 60
 $EndSheet
 $Sheet
-S 1700 2450 2650 900
+S 4050 3950 2600 950
+U 58D292AC
+F0 "5V" 60
+F1 "5V.sch" 60
+F2 "VCC" I R 6650 4150 60
+F3 "+5V" O L 4050 4200 60
+F4 "GND" I L 4050 4700 60
+$EndSheet
+$Sheet
+S 3950 6450 2500 900
+U 58D2C80A
+F0 "12V" 60
+F1 "12V.sch" 60
+F2 "GND" I L 3950 7150 60
+F3 "+12V" O L 3950 6650 60
+F4 "VCC" I R 6450 6700 60
+$EndSheet
+$Comp
+L PWR_FLAG #FLG01
+U 1 1 58DD0709
+P 3950 7550
+F 0 "#FLG01" H 3950 7645 50  0001 C CNN
+F 1 "PWR_FLAG" H 3950 7730 50  0000 C CNN
+F 2 "" H 3950 7550 50  0000 C CNN
+F 3 "" H 3950 7550 50  0000 C CNN
+	1    3950 7550
+	0    -1   -1   0
+$EndComp
+$Sheet
+S 4050 2700 2650 900
 U 58D2868B
 F0 "3,3V" 60
 F1 "3,3V.sch" 60
-F2 "VCC" I L 1700 2650 60
-F3 "+3,3V" O R 4350 2600 60
-F4 "GND" O L 1700 3150 60
+F2 "GND" O L 4050 3400 60
+F3 "VCC" I R 6700 2850 60
+F4 "+3,3V" O L 4050 2950 60
 $EndSheet
+Entry Wire Line
+	2850 2750 2950 2850
+Entry Wire Line
+	2850 4100 2950 4200
+Entry Wire Line
+	2850 5300 2950 5400
+Entry Wire Line
+	2850 6550 2950 6650
+$Comp
+L GND #PWR02
+U 1 1 59453698
+P 4100 7600
+F 0 "#PWR02" H 4100 7350 50  0001 C CNN
+F 1 "GND" H 4100 7450 50  0000 C CNN
+F 2 "" H 4100 7600 50  0000 C CNN
+F 3 "" H 4100 7600 50  0000 C CNN
+	1    4100 7600
+	1    0    0    -1
+$EndComp
+Connection ~ 5200 8700
+Wire Wire Line
+	5200 8700 5200 9300
+Wire Wire Line
+	6850 1150 6950 1150
+Wire Wire Line
+	6950 1150 6950 6700
+Wire Wire Line
+	6950 2850 6700 2850
+Wire Wire Line
+	6950 4150 6650 4150
+Connection ~ 6950 2850
+Wire Wire Line
+	6950 5450 6600 5450
+Connection ~ 6950 4150
+Wire Wire Line
+	6950 6700 6450 6700
+Connection ~ 6950 5450
+Wire Bus Line
+	2850 2750 2850 7550
+Wire Bus Line
+	2850 7550 2900 7550
+Wire Wire Line
+	3950 6650 2950 6650
+Wire Wire Line
+	4000 5400 2950 5400
+Wire Wire Line
+	4050 4200 2950 4200
+Wire Wire Line
+	4050 2950 2950 2950
+Wire Wire Line
+	2950 2950 2950 2850
+Wire Wire Line
+	4050 2100 3400 2100
+Wire Wire Line
+	3400 2100 3400 7700
+Wire Wire Line
+	3400 7700 3950 7700
+Wire Wire Line
+	3950 7150 3400 7150
+Connection ~ 3400 7150
+Wire Wire Line
+	4000 5950 3400 5950
+Connection ~ 3400 5950
+Wire Wire Line
+	4050 4700 3400 4700
+Connection ~ 3400 4700
+Wire Wire Line
+	4050 3400 3400 3400
+Connection ~ 3400 3400
+Wire Wire Line
+	3950 7700 3950 7550
+Wire Wire Line
+	4100 7600 3950 7600
+Connection ~ 3950 7600
 $Sheet
-S 1700 3700 2600 950
-U 58D292AC
-F0 "5V" 60
-F1 "5V.sch" 60
-F2 "VCC" I L 1700 3950 60
-F3 "+5V" O R 4300 3850 60
-F4 "GND" I L 1700 4400 60
-$EndSheet
-$Sheet
-S 1650 4950 2600 950
+S 4000 5200 2600 950
 U 58D2A118
 F0 "9V" 60
 F1 "9V.sch" 60
-F2 "+9V" O R 4250 5200 60
-F3 "GND" I L 1650 5700 60
-F4 "VCC" I L 1650 5150 60
+F2 "GND" I L 4000 5950 60
+F3 "+9V" O L 4000 5400 60
+F4 "VCC" I R 6600 5450 60
 $EndSheet
-$Sheet
-S 1650 6200 2500 900
-U 58D2C80A
-F0 "12V" 60
-F1 "12V.sch" 60
-F2 "+12V" O R 4150 6400 60
-F3 "GND" I L 1650 6900 60
-F4 "VCC" I L 1650 6400 60
-$EndSheet
+Entry Wire Line
+	2750 7250 2850 7150
+Entry Wire Line
+	2750 7350 2850 7250
+Entry Wire Line
+	2750 7450 2850 7350
+Entry Wire Line
+	2750 7550 2850 7450
+Wire Wire Line
+	2750 7250 2400 7250
+Wire Wire Line
+	2750 7350 2400 7350
+Wire Wire Line
+	2750 7450 2400 7450
+Wire Wire Line
+	2750 7550 2400 7550
+Wire Wire Line
+	3500 1100 4050 1100
+Wire Wire Line
+	3500 1100 3500 1150
 $Comp
-L GND #PWR01
-U 1 1 58D2DFDC
-P 1200 7450
-F 0 "#PWR01" H 1200 7200 50  0001 C CNN
-F 1 "GND" H 1200 7300 50  0000 C CNN
-F 2 "" H 1200 7450 50  0000 C CNN
-F 3 "" H 1200 7450 50  0000 C CNN
-	1    1200 7450
-	1    0    0    -1
-$EndComp
-Wire Wire Line
-	1700 950  850  950
-Wire Wire Line
-	850  950  850  6400
-Wire Wire Line
-	900  2650 1750 2650
-Wire Wire Line
-	850  3950 1700 3950
-Connection ~ 850  2650
-Wire Wire Line
-	850  5150 1650 5150
-Connection ~ 850  3950
-Wire Wire Line
-	850  6400 1650 6400
-Connection ~ 850  5150
-Wire Wire Line
-	1200 6850 1200 7450
-Connection ~ 1200 3100
-Connection ~ 1200 4400
-Wire Wire Line
-	1200 6900 1650 6900
-Connection ~ 1200 5700
-Connection ~ 1200 6850
-$Comp
-L PWR_FLAG #FLG?
-U 1 1 58DD06A1
-P 1200 950
-F 0 "#FLG?" H 1200 1045 50  0001 C CNN
-F 1 "PWR_FLAG" H 1200 1130 50  0000 C CNN
-F 2 "" H 1200 950 50  0000 C CNN
-F 3 "" H 1200 950 50  0000 C CNN
-	1    1200 950
+L PWR_FLAG #FLG03
+U 1 1 5945CAFB
+P 3500 1100
+F 0 "#FLG03" H 3500 1195 50  0001 C CNN
+F 1 "PWR_FLAG" H 3500 1280 50  0000 C CNN
+F 2 "" H 3500 1100 50  0000 C CNN
+F 3 "" H 3500 1100 50  0000 C CNN
+	1    3500 1100
 	1    0    0    -1
 $EndComp
 $Comp
-L PWR_FLAG #FLG?
-U 1 1 58DD0709
-P 1200 7400
-F 0 "#FLG?" H 1200 7495 50  0001 C CNN
-F 1 "PWR_FLAG" H 1200 7580 50  0000 C CNN
-F 2 "" H 1200 7400 50  0000 C CNN
-F 3 "" H 1200 7400 50  0000 C CNN
-	1    1200 7400
-	0    -1   -1   0
+L CONN_01X04 P2
+U 1 1 5945AFE9
+P 2200 7400
+F 0 "P2" H 2200 7650 50  0000 C CNN
+F 1 "CONN_01X04" V 2300 7400 50  0000 C CNN
+F 2 "" H 2200 7400 50  0000 C CNN
+F 3 "" H 2200 7400 50  0000 C CNN
+	1    2200 7400
+	-1   0    0    1
 $EndComp
+Text Label 3650 6650 2    60   ~ 0
+1
+Text Label 3750 5400 2    60   ~ 0
+2
+Text Label 3850 4200 0    60   ~ 0
+3
+Text Label 3700 2950 0    60   ~ 0
+4
+Text Label 2500 7250 0    60   ~ 0
+4
+Text Label 2550 7350 0    60   ~ 0
+3
+Text Label 2550 7450 0    60   ~ 0
+2
+Text Label 2600 7550 0    60   ~ 0
+1
 $EndSCHEMATC
