File: Single_transistor_AMP/_saved_Single_transistor_AMP.sch (KiCad schematic (older format))
At the start: 10 parts, among them P1 Signal_IN, P2 Signal_OUT, Q1 BC547

Commit message: single_amp
Parts:
- C2: footprint Capacitors_SMD:CP_Elec_4x5.7 -> Capacitors_THT:CP_Axial_L10.0mm_D4.5mm_P15.00mm_Horizontal
- Q1: footprint TO-92 -> TO_SOT_Packages_THT:TO-92_Inline_Narrow_Oval
- gave numbers to parts that had none: 1
- renumbered R2 to R1
Changed lines of the file:
@@
 F 0 "Q1" H 6100 4975 50  0000 L CNN
 F 1 "BC547" H 6100 4900 50  0000 L CNN
-F 2 "TO-92" H 6100 4825 50  0001 L CIN
+F 2 "TO_SOT_Packages_THT:TO-92_Inline_Narrow_Oval" H 6100 4825 50  0001 L CIN
 F 3 "https://www.fairchildsemi.com/datasheets/BC/BC546.pdf" H 5900 4900 50  0001 L CNN
 	1    5900 4900
@@
 F 0 "C2" H 6425 5850 50  0000 L CNN
 F 1 "22uF" H 6425 5650 50  0000 L CNN
-F 2 "Capacitors_SMD:CP_Elec_4x5.7" H 6438 5600 50  0001 C CNN
+F 2 "Capacitors_THT:CP_Axial_L10.0mm_D4.5mm_P15.00mm_Horizontal" H 6438 5600 50  0001 C CNN
 F 3 "https://industrial.panasonic.com/cdbs/www-data/pdf/RDE0000/ABA0000C1145.pdf" H 6400 5750 50  0001 C CNN
 	1    6400 5750
@@
 $EndComp
 $Comp
-L R R2
+L R R1
 U 1 1 58D92CE6
 P 5300 5450
-F 0 "R2" V 5380 5450 50  0000 C CNN
+F 0 "R1" V 5380 5450 50  0000 C CNN
 F 1 "1K" V 5300 5450 50  0000 C CNN
 F 2 "Resistors_THT:R_Axial_DIN0207_L6.3mm_D2.5mm_P15.24mm_Horizontal" V 5230 5450 50  0001 C CNN
@@
 Connection ~ 7100 4000
 $Comp
-L CONN_01X02 P?
+L CONN_01X02 P3
 U 1 1 59144AD5
 P 8150 5150
-F 0 "P?" H 8150 5300 50  0000 C CNN
+F 0 "P3" H 8150 5300 50  0000 C CNN
 F 1 "CONN_01X02" V 8250 5150 50  0000 C CNN
 F 2 "" H 8150 5150 50  0000 C CNN
