File: Single_transistor_AMP/Single_transistor_AMP.sch (KiCad schematic (older format))
At the start: 9 parts, among them P1 Signal_IN, P2 Signal_OUT, Q1 BC547

Commit message: single_amp
Parts:
- added P3: CONN_01X02, symbol CONN_01X02
- C2: footprint Capacitors_SMD:CP_Elec_4x5.7 -> Capacitors_THT:CP_Axial_L10.0mm_D4.5mm_P15.00mm_Horizontal
- renumbered R2 to R1
Changed lines of the file:
@@
 F 0 "C2" H 6425 5850 50  0000 L CNN
 F 1 "22uF" H 6425 5650 50  0000 L CNN
-F 2 "Capacitors_SMD:CP_Elec_4x5.7" H 6438 5600 50  0001 C CNN
+F 2 "Capacitors_THT:CP_Axial_L10.0mm_D4.5mm_P15.00mm_Horizontal" H 6438 5600 50  0001 C CNN
 F 3 "https://industrial.panasonic.com/cdbs/www-data/pdf/RDE0000/ABA0000C1145.pdf" H 6400 5750 50  0001 C CNN
 	1    6400 5750
@@
 $EndComp
 $Comp
-L GND #PWR01
+L GND #PWR1
 U 1 1 58D3C260
 P 6000 6400
-F 0 "#PWR01" H 6000 6150 50  0001 C CNN
+F 0 "#PWR1" H 6000 6150 50  0001 C CNN
 F 1 "GND" H 6000 6250 50  0000 C CNN
 F 2 "" H 6000 6400 50  0000 C CNN
@@
 $EndComp
 $Comp
-L R R2
+L R R1
 U 1 1 58D92CE6
 P 5300 5450
-F 0 "R2" V 5380 5450 50  0000 C CNN
+F 0 "R1" V 5380 5450 50  0000 C CNN
 F 1 "1K" V 5300 5450 50  0000 C CNN
 F 2 "Resistors_THT:R_Axial_DIN0207_L6.3mm_D2.5mm_P15.24mm_Horizontal" V 5230 5450 50  0001 C CNN
@@
 P 6000 4150
 F 0 "RL1" V 6080 4150 50  0000 C CNN
-F 1 "22K" V 6000 4150 50  0000 C CNN
+F 1 "22K" V 6000 4150 50  0001 C CNN
 F 2 "Resistors_THT:R_Axial_DIN0207_L6.3mm_D2.5mm_P15.24mm_Horizontal" V 5930 4150 50  0001 C CNN
 F 3 "https://www.seielect.com/Catalog/SEI-CF_CFM.pdf" H 6000 4150 50  0001 C CNN
@@
 $EndComp
 $Comp
-L PWR_FLAG #FLG02
+L PWR_FLAG #FLG2
 U 1 1 58D949EB
 P 7400 4000
-F 0 "#FLG02" H 7400 4095 50  0001 C CNN
+F 0 "#FLG2" H 7400 4095 50  0001 C CNN
 F 1 "PWR_FLAG" H 7400 4180 50  0000 C CNN
 F 2 "" H 7400 4000 50  0000 C CNN
@@
 $EndComp
 $Comp
-L +12V #PWR03
+L +12V #PWR2
 U 1 1 58DC2C33
 P 7100 3900
-F 0 "#PWR03" H 7100 3750 50  0001 C CNN
+F 0 "#PWR2" H 7100 3750 50  0001 C CNN
 F 1 "+12V" H 7100 4040 50  0000 C CNN
 F 2 "" H 7100 3900 50  0000 C CNN
@@
 $EndComp
 $Comp
-L PWR_FLAG #FLG04
+L PWR_FLAG #FLG1
 U 1 1 58DC2D79
 P 7150 6100
-F 0 "#FLG04" H 7150 6195 50  0001 C CNN
+F 0 "#FLG1" H 7150 6195 50  0001 C CNN
 F 1 "PWR_FLAG" H 7150 6280 50  0000 C CNN
 F 2 "" H 7150 6100 50  0000 C CNN
@@
 	7100 3900 7100 4000
 Connection ~ 7100 4000
+$Comp
+L CONN_01X02 P3
+U 1 1 59144AD5
+P 8150 5150
+F 0 "P3" H 8150 5300 50  0000 C CNN
+F 1 "CONN_01X02" V 8250 5150 50  0000 C CNN
+F 2 "" H 8150 5150 50  0000 C CNN
+F 3 "" H 8150 5150 50  0000 C CNN
+	1    8150 5150
+	1    0    0    -1
+$EndComp
 $EndSCHEMATC

Commit message: Kursa_darbs_PCB
Parts:
- Q1: footprint TO-92 -> TO_SOT_Packages_THT:TO-92_Inline_Narrow_Oval
Changed lines of the file:
@@
 F 0 "Q1" H 6100 4975 50  0000 L CNN
 F 1 "BC547" H 6100 4900 50  0000 L CNN
-F 2 "TO-92" H 6100 4825 50  0001 L CIN
+F 2 "TO_SOT_Packages_THT:TO-92_Inline_Narrow_Oval" H 6100 4825 50  0001 L CIN
 F 3 "https://www.fairchildsemi.com/datasheets/BC/BC546.pdf" H 5900 4900 50  0001 L CNN
 	1    5900 4900
@@
 $EndComp
 $Comp
-L GND #PWR1
+L GND #PWR01
 U 1 1 58D3C260
 P 6000 6400
-F 0 "#PWR1" H 6000 6150 50  0001 C CNN
+F 0 "#PWR01" H 6000 6150 50  0001 C CNN
 F 1 "GND" H 6000 6250 50  0000 C CNN
 F 2 "" H 6000 6400 50  0000 C CNN
@@
 $EndComp
 $Comp
-L PWR_FLAG #FLG2
+L PWR_FLAG #FLG02
 U 1 1 58D949EB
 P 7400 4000
-F 0 "#FLG2" H 7400 4095 50  0001 C CNN
+F 0 "#FLG02" H 7400 4095 50  0001 C CNN
 F 1 "PWR_FLAG" H 7400 4180 50  0000 C CNN
 F 2 "" H 7400 4000 50  0000 C CNN
@@
 $EndComp
 $Comp
-L +12V #PWR2
+L +12V #PWR03
 U 1 1 58DC2C33
 P 7100 3900
-F 0 "#PWR2" H 7100 3750 50  0001 C CNN
+F 0 "#PWR03" H 7100 3750 50  0001 C CNN
 F 1 "+12V" H 7100 4040 50  0000 C CNN
 F 2 "" H 7100 3900 50  0000 C CNN
@@
 $EndComp
 $Comp
-L PWR_FLAG #FLG1
+L PWR_FLAG #FLG04
 U 1 1 58DC2D79
 P 7150 6100
-F 0 "#FLG1" H 7150 6195 50  0001 C CNN
+F 0 "#FLG04" H 7150 6195 50  0001 C CNN
 F 1 "PWR_FLAG" H 7150 6280 50  0000 C CNN
 F 2 "" H 7150 6100 50  0000 C CNN
